File: Hardware/PlantWateringDevice/DataHandling.kicad_sch (KiCad schematic)
At the start: 13 parts, among them J1 Conn_02x04_Counter_Clockwise, J5 Conn_02x03_Odd_Even, SW1 SW_DIP_x02, SW3 SW_Push, SW4 SW_DIP_x02, SW7 SW_DIP_x02, U4 PIC10F202-IOT

Commit message: firmware implementation
Other:
- note added: "CHANGE NAME ITS CONFUSING HUMIDITY_SENSOR_COMP HUMIDITY_SENSOR_OUT"
- note added: "GP3 (Pin 6) - Input-only"
- note added: "LESS SWITECHES"
- note added: "RST 4017 BUTTON AFTER PROGRAMMING"
- note removed: "GP3 (Pin 6) - Input-only Either data from Humidity Sensor or selection of watering periodicity from push button"
Changed lines of the file:
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@@
 			(font
 				(size 1.27 1.27)
+				(thickness 0.254)
+				(bold yes)
 			)
 		)
 	)
-	(text "GP3 (Pin 6) - Input-only\nEither data from Humidity\nSensor or selection of\nwatering periodicity from\npush button"
+	(text "LESS SWITECHES"
 		(exclude_from_sim no)
-		(at 166.116 55.118 0)
+		(at 255.27 53.086 0)
+		(effects
+			(font
+				(size 5.08 5.08)
+				(thickness 1.27)
+				(bold yes)
+			)
+		)
+	)
+	(text "GP3 (Pin 6) - Input-only\n"
+		(exclude_from_sim no)
+		(at 160.528 66.294 0)
 		(effects
 			(font
@@
 			(font
 				(size 1.27 1.27)
+				(thickness 0.254)
+				(bold yes)
+			)
+		)
+	)
+	(text "RST 4017 BUTTON AFTER PROGRAMMING"
+		(exclude_from_sim no)
+		(at 223.774 40.64 0)
+		(effects
+			(font
+				(size 5.08 5.08)
+				(thickness 1.27)
+				(bold yes)
 			)
 		)
@@
 			(font
 				(size 1.27 1.27)
+				(thickness 0.254)
+				(bold yes)
 			)
 		)
+	)
+	(text "CHANGE NAME ITS CONFUSING\n\nHUMIDITY_SENSOR_COMP\nHUMIDITY_SENSOR_OUT"
+		(exclude_from_sim no)
+		(at 235.712 114.808 0)
+		(effects
+			(font
+				(size 5.08 5.08)
+				(thickness 1.27)
+				(bold yes)
+			)
+		)
