File: Hardware/PlantWateringDevice/HumiditySensor.kicad_sch (KiCad schematic)
At the start: 11 parts, among them U1 MCP6002-xSN

Commit message: firmware implementation
Other:
- note added: "LED TO TP2 pzelaczniki foopriny"
- note added: "POSITIVE FEEDBACK"
Changed lines of the file:
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@@
 	(generator_version "9.0")
 	(paper "A4")
+	(text "LED TO TP2 pzelaczniki foopriny"
+		(exclude_from_sim no)
+		(at 171.196 46.228 0)
+		(effects
+			(font
+				(size 5.08 5.08)
+				(thickness 1.27)
+				(bold yes)
+			)
+		)
+	)
+	(text "POSITIVE FEEDBACK"
+		(exclude_from_sim no)
+		(at 153.416 132.842 0)
+		(effects
+			(font
+				(size 5.08 5.08)
+				(thickness 1.27)
+				(bold yes)
+			)
+		)
+	)
 	(text "Potentiometer is not mount on PCB"
 		(exclude_from_sim no)

Commit message: fix in algo
Parts:
- R3: now not fitted; now left out of the parts list
Changed lines of the file:
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@@
 	(text "LED TO TP2 pzelaczniki foopriny"
 		(exclude_from_sim no)
-		(at 171.196 46.228 0)
+		(at 201.676 20.32 0)
 		(effects
 			(font
@@
 		(at 118.11 80.01 90)
 		(unit 1)
-		(exclude_from_sim no)
-		(in_bom yes)
-		(on_board yes)
-		(dnp no)
+		(exclude_from_sim yes)
+		(in_bom no)
+		(on_board no)
+		(dnp yes)
 		(fields_autoplaced yes)
 		(property "Reference" "R3"
