File: Hardware/PlantWateringDevice/Display.kicad_sch (KiCad schematic)
At the start: 24 parts, among them SW2 SW_Push, U1 MCP6002-xSN, U2 74LVC1G3157, U6 74HC74, U7 74HC4017D

Commit message: firmware implementation
Parts:
- R31, R32: value 220R -> 510R
- R47: value 220R -> 120R
Changed lines of the file:
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@@
 			)
 		)
-		(property "Value" "220R"
+		(property "Value" "510R"
 			(at 128.27 93.9799 0)
 			(effects
@@
 		(fields_autoplaced yes)
 		(property "Reference" "R31"
-			(at 128.27 62.2299 0)
-			(effects
-				(font
-					(size 1.27 1.27)
-				)
-				(justify left)
-			)
-		)
-		(property "Value" "220R"
-			(at 128.27 64.7699 0)
-			(effects
-				(font
-					(size 1.27 1.27)
-				)
-				(justify left)
+			(at 123.19 62.2299 0)
+			(effects
+				(font
+					(size 1.27 1.27)
+				)
+				(justify right)
+			)
+		)
+		(property "Value" "510R"
+			(at 123.19 64.7699 0)
+			(effects
+				(font
+					(size 1.27 1.27)
+				)
+				(justify right)
 			)
 		)
@@
 			)
 		)
-		(property "Value" "220R"
+		(property "Value" "120R"
 			(at 246.38 121.9199 0)
 			(effects

Commit message: fix #29, fix #31
Connections:
- net DISPLAY_DATA renamed LCD_DATA
- net HUMIDITY_SENSOR_COMP renamed POTENTIOMETER_DATA
- net HUMIDITY_SENSOR_IN renamed HUMIDITY_SENSOR
Changed lines of the file:
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@@
 		)
 	)
-	(global_label "DISPLAY_DATA"
+	(global_label "LCD_DATA"
 		(shape output)
 		(at 144.78 31.75 0)
@@
 		)
 		(property "Intersheetrefs" "${INTERSHEET_REFS}"
-			(at 160.7072 31.75 0)
+			(at 156.7157 31.75 0)
 			(effects
 				(font
@@
 		)
 	)
-	(global_label "HUMIDITY_SENSOR_COMP"
+	(global_label "POTENTIOMETER_DATA"
 		(shape input)
 		(at 100.33 26.67 180)
@@
 		)
 		(property "Intersheetrefs" "${INTERSHEET_REFS}"
-			(at 73.9405 26.67 0)
+			(at 77.0249 26.67 0)
 			(effects
 				(font
@@
 		)
 	)
-	(global_label "HUMIDITY_SENSOR_IN"
+	(global_label "HUMIDITY_SENSOR"
 		(shape input)
 		(at 100.33 36.83 180)
@@
 		)
 		(property "Intersheetrefs" "${INTERSHEET_REFS}"
-			(at 77.3271 36.83 0)
+			(at 80.23 36.83 0)
 			(effects
 				(font
