File: Hardware/PlantWateringDevice/Mechanic.kicad_sch (KiCad schematic)
At the start: 4 parts

Commit message: fixes before sending pcb and 3d model to production
Parts:
- H1, H2, H3, H4: footprint MountingHole:MountingHole_3.5mm_Pad -> MountingHole:MountingHole_3mm_Pad
Changed lines of the file:
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@@
 			)
 		)
-		(property "Footprint" "MountingHole:MountingHole_3.5mm_Pad"
+		(property "Footprint" "MountingHole:MountingHole_3mm_Pad"
 			(at 77.47 101.6 0)
 			(effects
@@
 			)
 		)
-		(property "Footprint" "MountingHole:MountingHole_3.5mm_Pad"
+		(property "Footprint" "MountingHole:MountingHole_3mm_Pad"
 			(at 102.87 102.87 0)
 			(effects
@@
 			)
 		)
-		(property "Footprint" "MountingHole:MountingHole_3.5mm_Pad"
+		(property "Footprint" "MountingHole:MountingHole_3mm_Pad"
 			(at 77.47 83.82 0)
 			(effects
@@
 			)
 		)
-		(property "Footprint" "MountingHole:MountingHole_3.5mm_Pad"
+		(property "Footprint" "MountingHole:MountingHole_3mm_Pad"
 			(at 102.87 83.82 0)
 			(effects

Commit message: fix #16, fix #17, fix #18, fix #19, fix #20, fix #26, fix #27, fix #28, fix #30, fix #32, fix#33, fix #34, fix #35, fix #38
Parts:
- H1, H2, H3, H4: footprint MountingHole:MountingHole_3mm_Pad -> MountingHole:MountingHole_2.5mm_Pad
