File: Hardware/PlantWateringDevice/PowerManagement.kicad_sch (KiCad schematic)
At the start: 15 parts, among them J1 USB_B_Micro, M1 Motor_DC, Q1 AO3404A

Commit message: change pcb stackup
Parts:
- renumbered C14/25V1 to C14
Changed lines of the file:
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@@
 		(in_pos_files yes)
 		(dnp no)
-		(property "Reference" "C14/25V1"
+		(property "Reference" "C14"
 			(at 171.831 87.7316 0)
 			(show_name no)
@@
 			(project "PlantWateringDevice"
 				(path "/1ef241b3-83d7-48ae-bcca-b7d0eea44e63/a141cb94-983c-4780-96e1-70ed49312478"
-					(reference "C14/25V1")
+					(reference "C14")
 					(unit 1)
 				)
